Commit message: Fixed bugs and created demo with real robot

File: iiwa_stack-master/iiwa_description/urdf/iiwa_robotiq.urdf.xacro (robot description, xacro)
@@ -37,5 +37,5 @@
       <parent link="iiwa_link_ee"/>
       <child link="robotiq_coupler"/>
-      <origin xyz="0 0 0" rpy="0 0 0"/>
+      <origin xyz="0 0 0.03" rpy="0 0 0"/>
     </joint>
   <!-- <xacro:robotiq_arg2f_85_model></xacro:robotiq_arg2f_85_model> -->

File: iiwa_stack-master/iiwa_description/urdf/iiwa_robotiq_cam.urdf.xacro (robot description, xacro)
@@ -25,5 +25,5 @@
       </visual>
       <collision>
-        <origin xyz="0 0 0.01" rpy="0 0 0"/>
+        <origin xyz="0 0 0" rpy="0 0 0"/>
         <geometry>
           <mesh
@@ -36,5 +36,5 @@
     <parent link="iiwa_link_ee"/>
     <child link="camera_link"/>
-    <origin xyz="0 0 0.010" rpy="1.5708 0 0"/>
+    <origin xyz="0 0 0.04" rpy="1.5708 0 0"/>
   </joint>
   <joint name="camera_to_robotiq" type="fixed">

File: iiwa_stack-master/iiwa_description/urdf/iiwa_zimmer.urdf.xacro (robot description, xacro)
@@ -20,5 +20,5 @@
     <parent link="iiwa_link_ee"/>
     <child link="GEP5006IO-00-A(0)"/>
-    <origin xyz="0 0 0.01" rpy="0 0 0"/>
+    <origin xyz="0 0 0.03" rpy="0 0 0"/>
   </joint>
 </robot>
